Commit message: Add depth camera

File: gazebo_demo/urdf/ABot.urdf.xacro (robot description, xacro)
@@ -334,5 +334,79 @@
       </plugin>
     </sensor>
-  </gazebo>
+ </gazebo>
+<!-- Depth Camera -->
+<link name="depth_camera_link">
+    <collision>
+      <origin xyz="0 0 0" rpy="0 0 0"/>
+      <geometry>
+    <box size="0.01 0.01 0.01"/>
+      </geometry>
+    </collision>
+    <visual>
+      <origin xyz="0 0 0" rpy="0 0 0"/>
+      <geometry>
+    <box size="0.01 0.01 0.01"/>
+      </geometry>
+      <material name="blue"/>
+    </visual>
+    <inertial>
+      <mass value="1e-5" />
+      <origin xyz="0 0 0" rpy="0 0 0"/>
+      <inertia ixx="1e-6" ixy="0" ixz="0" iyy="1e-6" iyz="0" izz="1e-6" />
+    </inertial>
+  </link>
+<gazebo reference="depth_camera_link">
+    <material>Gazebo/Black</material>
+    <mu1>0.000001</mu1>
+    <mu2>0.000001</mu2>
+  </gazebo>
+<joint name="depth_camera_joint" type="fixed">
+    <axis xyz="0 0 0" />
+    <origin xyz="0.2 0 0.15" rpy="0 0 0"/>
+    <parent link="base_link"/>
+    <child link="depth_camera_link"/>
+  </joint>
+<gazebo reference="depth_camera_link">
+  <sensor name="depth_camera" type="depth">
+    <update_rate>20</update_rate>
+    <camera>
+      <horizontal_fov>1.047198</horizontal_fov>
+      <image>
+        <width>640</width>
+        <height>480</height>
+        <format>R8G8B8</format>
+      </image>
+      <clip>
+        <near>0.05</near>
+        <far>3</far>
+      </clip>
+    </camera>
+    <plugin name="depth_camera_controller" filename="libgazebo_ros_openni_kinect.so">
+      <baseline>0.2</baseline>
+      <alwaysOn>true</alwaysOn>
+      <updateRate>1.0</updateRate>
+      <cameraName>depth_camera_ir</cameraName>
+      <imageTopicName>/depth_camera/color/image_raw</imageTopicName>
+      <cameraInfoTopicName>/depth_camera/color/camera_info</cameraInfoTopicName>
+      <depthImageTopicName>/depth_camera/depth/image_raw</depthImageTopicName>
+      <depthImageInfoTopicName>/depth_camera/depth/camera_info</depthImageInfoTopicName>
+      <pointCloudTopicName>/depth_camera/depth/points</pointCloudTopicName>
+      <frameName>depth_camera_link</frameName>
+      <pointCloudCutoff>0.5</pointCloudCutoff>
+      <pointCloudCutoffMax>3.0</pointCloudCutoffMax>
+      <distortionK1>0.00000001</distortionK1>
+      <distortionK2>0.00000001</distortionK2>
+      <distortionK3>0.00000001</distortionK3>
+      <distortionT1>0.00000001</distortionT1>
+      <distortionT2>0.00000001</distortionT2>
+      <CxPrime>0</CxPrime>
+      <Cx>0</Cx>
+      <Cy>0</Cy>
+      <focalLength>0</focalLength>
+      <hackBaseline>0</hackBaseline>
+    </plugin>
+  </sensor>
+</gazebo>
+<!-- ____________ -->
 <gazebo>
   <plugin name="differential_drive_controller" filename="libgazebo_ros_diff_drive.so">

Commit message: Add train model and update

File: gazebo_demo/urdf/ABot.urdf.xacro (robot description, xacro)
@@ -63,5 +63,5 @@
   <inertial>
     <origin rpy="1.5707963267948966 0 0" xyz="0 0 0" />
-    <mass value="0.1" />
+    <mass value="0.5" />
     <inertia  ixx="0.01" ixy="0.0"  ixz="0.0"  iyy="0.01"  iyz="0.0"  izz="0.01" />
   </inertial>
@@ -101,5 +101,5 @@
   <inertial>
     <origin rpy="1.5707963267948966 0 0" xyz="0 0 0" />
-    <mass value="0.1" />
+    <mass value="0.5" />
     <inertia  ixx="0.01" ixy="0.0"  ixz="0.0"  iyy="0.01"  iyz="0.0"  izz="0.01" />
   </inertial>
@@ -379,5 +379,5 @@
       <clip>
         <near>0.05</near>
-        <far>3</far>
+        <far>10</far>
       </clip>
     </camera>
@@ -394,5 +394,5 @@
       <frameName>depth_camera_link</frameName>
       <pointCloudCutoff>0.5</pointCloudCutoff>
-      <pointCloudCutoffMax>3.0</pointCloudCutoffMax>
+      <pointCloudCutoffMax>5.0</pointCloudCutoffMax>
       <distortionK1>0.00000001</distortionK1>
       <distortionK2>0.00000001</distortionK2>

Commit message: Updata model
add second depth camera, updata train model

File: gazebo_demo/urdf/ABot.urdf.xacro (robot description, xacro)
@@ -385,5 +385,5 @@
       <baseline>0.2</baseline>
       <alwaysOn>true</alwaysOn>
-      <updateRate>1.0</updateRate>
+      <updateRate>20</updateRate>
       <cameraName>depth_camera_ir</cameraName>
       <imageTopicName>/depth_camera/color/image_raw</imageTopicName>
@@ -393,6 +393,80 @@
       <pointCloudTopicName>/depth_camera/depth/points</pointCloudTopicName>
       <frameName>depth_camera_link</frameName>
-      <pointCloudCutoff>0.5</pointCloudCutoff>
-      <pointCloudCutoffMax>5.0</pointCloudCutoffMax>
+      <pointCloudCutoff>0</pointCloudCutoff> <!-- change from 0.1 - 10.0 -->
+      <pointCloudCutoffMax>255</pointCloudCutoffMax>
+      <distortionK1>0.00000001</distortionK1>
+      <distortionK2>0.00000001</distortionK2>
+      <distortionK3>0.00000001</distortionK3>
+      <distortionT1>0.00000001</distortionT1>
+      <distortionT2>0.00000001</distortionT2>
+      <CxPrime>0</CxPrime>
+      <Cx>0</Cx>
+      <Cy>0</Cy>
+      <focalLength>0</focalLength>
+      <hackBaseline>0</hackBaseline>
+    </plugin>
+  </sensor>
+</gazebo>
+<!-- ____________ -->
+<!-- Depth Camera 2 -->
+<link name="depth_camera_link_2">
+    <collision>
+      <origin xyz="0 0 0" rpy="0 0 0"/>
+      <geometry>
+    <box size="0.01 0.01 0.01"/>
+      </geometry>
+    </collision>
+    <visual>
+      <origin xyz="0 0 0" rpy="0 0 0"/>
+      <geometry>
+    <box size="0.01 0.01 0.01"/>
+      </geometry>
+      <material name="blue"/>
+    </visual>
+    <inertial>
+      <mass value="1e-5" />
+      <origin xyz="0 0 0" rpy="0 0 0"/>
+      <inertia ixx="1e-6" ixy="0" ixz="0" iyy="1e-6" iyz="0" izz="1e-6" />
+    </inertial>
+  </link>
+<gazebo reference="depth_camera_link_2">
+    <material>Gazebo/Black</material>
+    <mu1>0.000001</mu1>
+    <mu2>0.000001</mu2>
+  </gazebo>
+<joint name="depth_camera_joint_2" type="fixed">
+    <axis xyz="0 0 0" />
+    <origin xyz="0.2 -0.05 0.175" rpy="0 0 0"/>
+    <parent link="base_link"/>
+    <child link="depth_camera_link_2"/>
+  </joint>
+<gazebo reference="depth_camera_link_2">
+  <sensor name="depth_camera_2" type="depth">
+    <update_rate>20</update_rate>
+    <camera>
+      <horizontal_fov>1.047198</horizontal_fov>
+      <image>
+        <width>640</width>
+        <height>480</height>
+        <format>R8G8B8</format>
+      </image>
+      <clip>
+        <near>0.05</near>
+        <far>10</far>
+      </clip>
+    </camera>
+    <plugin name="depth_camera_controller" filename="libgazebo_ros_openni_kinect.so">
+      <baseline>0.2</baseline>
+      <alwaysOn>true</alwaysOn>
+      <updateRate>20</updateRate>
+      <cameraName>depth_camera_ir_2</cameraName>
+      <imageTopicName>/depth_camera_2/color/image_raw</imageTopicName>
+      <cameraInfoTopicName>/depth_camera_2/color/camera_info</cameraInfoTopicName>
+      <depthImageTopicName>/depth_camera_2/depth/image_raw</depthImageTopicName>
+      <depthImageInfoTopicName>/depth_camera_2/depth/camera_info</depthImageInfoTopicName>
+      <pointCloudTopicName>/depth_camera_2/depth/points</pointCloudTopicName>
+      <frameName>depth_camera_link_2</frameName>
+      <pointCloudCutoff>0.1</pointCloudCutoff> <!-- change from 0.1 - 10.0 -->
+      <pointCloudCutoffMax>10.0</pointCloudCutoffMax>
       <distortionK1>0.00000001</distortionK1>
       <distortionK2>0.00000001</distortionK2>
